File: leds-8.sch (KiCad schematic (older format))
At the start: 16 parts

Commit message: Fix startup circuit
Use a zener-diode instead of just resistors.
This makes stuff much easier since it 'protects' the CPU from the high battery voltage.
Parts:
- C10, C11, C12, C13, C14, C15, C16, C9: value C -> 100n
