File: haargabel.sch (KiCad schematic (older format))
At the start: 36 parts, among them J1 SWD, J2 USB_B_Micro, J3 Conn_01x02, SW1 SW_Push, U1 ATSAML21E15B-MUT, U2 MCP73831-2-OT, U3 TPS79330-EP, U4 TPS22929D, U5 MPU-6050

Commit message: Fix startup circuit
Use a zener-diode instead of just resistors.
This makes stuff much easier since it 'protects' the CPU from the high battery voltage.
Parts:
- removed J3: Conn_01x02, Connector_PinHeader_2.54mm:PinHeader_1x02_P2.54mm_Vertical, symbol Connector_Generic:Conn_01x02
- removed R3: 470R, Resistor_SMD:R_0603_1608Metric, symbol Device:R
- added D26: BZT52C2V7T-7, Diode_SMD:D_SOD-523, symbol Device:D_Zener
- added J3: Conn_01x03, Connector_Molex:Molex_PicoBlade_53398-0371_1x03-1MP_P1.25mm_Vertical, symbol Connector_Generic:Conn_01x03
- added R10, R9: 270R, Resistor_SMD:R_0603_1608Metric, symbol Device:R
- R4: value 100k -> 1k
- SW1: value SW_Push -> SKRKAEE020
- gave numbers to parts that had none: 3
Connections:
- net +3V0: now also R9.1
- net +BATT: now also SW1.1, J3.1 (Pin_1); no longer SW1.2
- net GND: now also D26.2 (A), J3.3 (Pin_3); no longer D25.1 (K)
- net STAT: now also D25.1 (K); no longer R2.2
- net VBUS: now also R2.2
- net EN: now reaches U1.3 (PA02)
- net EN: now also R4.1, U3.3 (EN), D26.1 (K), R10.2, R9.2
- net PWR_ON: no longer names the net of U1.21 (PA22)
- new net: R10.1, SW1.2
Other:
- moved on the sheet: C25, C30, D25, J2, R1, R2, R4, R7, R8, SW1, U2

Commit message: Make it longer
Add two more LEDs, making the whole thing 30mm longer
Parts:
- removed H1, H2, H3: MountingHole, MountingHole:Mousebite_0.4_0.6, symbol Mechanical:MountingHole
Changed lines of the file:
@@
 S 8750 2400 600  500
 U 5C9BE103
-F0 "led8_1" 50
-F1 "leds-8.sch" 50
+F0 "led10_1" 50
+F1 "leds-10.sch" 50
 F2 "SDI" I L 8750 2500 50
 F3 "CKI" I L 8750 2600 50
@@
 S 9600 2400 600  500
 U 5C9BDF32
-F0 "led8_2" 50
-F1 "leds-8.sch" 50
+F0 "led10_2" 50
+F1 "leds-10.sch" 50
 F2 "SDI" I L 9600 2500 50
 F3 "CKI" I L 9600 2600 50
@@
 S 10450 2400 550  500
 U 5C9BE4CD
-F0 "led8_3" 50
-F1 "leds-8.sch" 50
+F0 "led10_3" 50
+F1 "leds-10.sch" 50
 F2 "SDI" I L 10450 2500 50
 F3 "CKI" I L 10450 2600 50
@@
 Connection ~ 5150 7000
 $Comp
-L Mechanical:MountingHole H1
-U 1 1 5CC63140
-P 650 600
-F 0 "H1" H 750 646 50  0000 L CNN
-F 1 "MountingHole" H 750 555 50  0000 L CNN
-F 2 "MountingHole:Mousebite_0.4_0.6" H 650 600 50  0001 C CNN
-F 3 "~" H 650 600 50  0001 C CNN
-	1    650  600
-	1    0    0    -1
-$EndComp
-$Comp
-L Mechanical:MountingHole H2
-U 1 1 5CC633E9
-P 650 800
-F 0 "H2" H 750 846 50  0000 L CNN
-F 1 "MountingHole" H 750 755 50  0000 L CNN
-F 2 "MountingHole:Mousebite_0.4_0.6" H 650 800 50  0001 C CNN
-F 3 "~" H 650 800 50  0001 C CNN
-	1    650  800
-	1    0    0    -1
-$EndComp
-$Comp
-L Mechanical:MountingHole H3
-U 1 1 5CC63447
-P 650 1000
-F 0 "H3" H 750 1046 50  0000 L CNN
-F 1 "MountingHole" H 750 955 50  0000 L CNN
-F 2 "MountingHole:Mousebite_0.4_0.6" H 650 1000 50  0001 C CNN
-F 3 "~" H 650 1000 50  0001 C CNN
-	1    650  1000
-	1    0    0    -1
-$EndComp
-$Comp
 L Device:R R9

Commit message: Re-Annotate, so the LED numbering makes more sense
Parts:
- renumbered C25 to C1, C34 to C10, C36 to C11, C37 to C12, C38 to C13, C35 to C14, C26 to C2, C27 to C3, C28 to C4, C30 to C5, C29 to C6, C31 to C7, C32 to C8, C33 to C9, D25 to D1, D26 to D2, R7 to R1, R8 to R2, R1 to R3, R2 to R4, R9 to R5, R4 to R6, R10 to R7, R5 to R8, R6 to R9, U5 to U4, U4 to U5
