File: leds-10.sch (KiCad schematic (older format))
At the start: 16 parts

Commit message: Make it longer
Add two more LEDs, making the whole thing 30mm longer
Parts:
- added C41, C42: 100n, Capacitor_SMD:C_0603_1608Metric, symbol Device:C
- added D29, D30: APA102-2020, LED_SMD:LED-APA102-2020, symbol LED:APA102-2020
Connections:
- net CKO: now also D30.2 (CKO); no longer D16.2 (CKO)
- net GND: now also C41.2, C42.2, D29.6 (GND), D30.6 (GND)
- net SDO: now also D30.3 (SDO); no longer D16.3 (SDO)
- net VCC: now also C41.1, C42.1, D29.1 (VDD), D30.1 (VDD)
- new net: D16.2 (CKO), D29.5 (CKI)
- new net: D16.3 (SDO), D29.4 (SDI)
- new net: D29.2 (CKO), D30.5 (CKI)
- new net: D29.3 (SDO), D30.4 (SDI)

Commit message: Re-Annotate, so the LED numbering makes more sense
Parts:
- renumbered C9 to C25, C10 to C26, C11 to C27, C12 to C28, C13 to C29, C14 to C30, C15 to C31, C16 to C32, C41 to C33, C42 to C34, D9 to D13, D10 to D14, D11 to D15, D12 to D16, D13 to D17, D14 to D18, D15 to D19, D16 to D20, D29 to D21, D30 to D22
